Commit message: left wheel and joint added

File: src/my_robot/urdf/my_robot.xacro (robot description, xacro)
@@ -7,30 +7,4 @@
     <child link="chassis" />
   </joint>
-<!--
-  <link name="left_wheel">
-    <pose>10 0 0 0 0 0</pose>
-    <inertial>
-      <mass value="5.0" />
-      <origin xyz="0 0 0" rpy="0 1.5707 1.5707" />
-      <inertia
-        ixx="0.1" ixy="0" ixz="0"
-        iyy="0.1" iyz="0"
-        izz="0.1"
-      />
-    </inertial>
-    <collision name="collision">
-      <origin xyz="0 0 0" rpy="0 1.5707 1.5707" />
-      <geometry>
-        <cylinder radius="0.1" length="0.05" />
-      </geometry>
-    </collision>
-    <visual name="visual">
-      <origin xyz="0 0 0" rpy="0 1.5707 1.5707" />
-      <geometry>
-        <cylinder radius="0.1" length="0.05" />
-      </geometry>
-    </visual>
-  </link>
--->
   <link name="chassis">
     <pose>0 0 0.1 0 0 0</pose>
@@ -104,3 +78,35 @@
     </visual>
   </link>
+  <link name="left_wheel">
+    <pose>10 0 0 0 0 0</pose>
+    <inertial>
+      <mass value="5.0" />
+      <origin xyz="0 0 0" rpy="0 1.5707 1.5707" />
+      <inertia
+        ixx="0.1" ixy="0" ixz="0"
+        iyy="0.1" iyz="0"
+        izz="0.1"
+      />
+    </inertial>
+    <collision name="collision">
+      <origin xyz="0 0 0" rpy="0 1.5707 1.5707" />
+      <geometry>
+        <cylinder radius="0.1" length="0.05" />
+      </geometry>
+    </collision>
+    <visual name="visual">
+      <origin xyz="0 0 0" rpy="0 1.5707 1.5707" />
+      <geometry>
+        <cylinder radius="0.1" length="0.05" />
+      </geometry>
+    </visual>
+  </link>
+  <joint type="continuous" name="left_wheel_hinge">
+    <origin xyz="0 0.15 0" rpy="0 0 0" />
+    <child link="left_wheel" />
+    <parent link="chassis" />
+    <axis xyz="0 1 0" rpy="0 0 0" />
+    <limit effort="10000" velocity="1000" />
+    <dynamics damping="1.0" friction="1.0" />
+  </joint>
 </robot>

Commit message: right wheel and joint added

File: src/my_robot/urdf/my_robot.xacro (robot description, xacro)
@@ -55,29 +55,5 @@
     </visual>
   </link>
-  <link name="camera">
-    <inertial>
-      <mass value="0.1" />
-      <origin xyz="0 0 0" rpy="0 0 0" />
-      <inertia
-        ixx="0.1" ixy="0" ixz="0"
-        iyy="1e-6" iyz="0"
-        izz="1e-6"
-      />
-    </inertial>
-    <collision name="camera_collision">
-      <origin xyz="0 0 0" rpy="0 0 0" />
-      <geometry>
-        <box size="0.05 0.05 0.05" />
-      </geometry>
-    </collision>
-    <visual name="camera_visual">
-      <origin xyz="0 0 0" rpy="0 0 0" />
-      <geometry>
-        <box size="0.05 0.05 0.05" />
-      </geometry>
-    </visual>
-  </link>
   <link name="left_wheel">
-    <pose>10 0 0 0 0 0</pose>
     <inertial>
       <mass value="5.0" />
@@ -89,5 +65,5 @@
       />
     </inertial>
-    <collision name="collision">
+    <collision name="left_wheel_collision">
       <origin xyz="0 0 0" rpy="0 1.5707 1.5707" />
       <geometry>
@@ -95,5 +71,5 @@
       </geometry>
     </collision>
-    <visual name="visual">
+    <visual name="left_wheel_visual">
       <origin xyz="0 0 0" rpy="0 1.5707 1.5707" />
       <geometry>
@@ -110,3 +86,34 @@
     <dynamics damping="1.0" friction="1.0" />
   </joint>
+  <link name="right_wheel">
+    <inertial>
+      <mass value="5.0" />
+      <origin xyz="0 0 0" rpy="0 1.5707 1.5707" />
+      <inertia
+        ixx="0.1" ixy="0" ixz="0"
+        iyy="0.1" iyz="0"
+        izz="0.1"
+      />
+    </inertial>
+    <collision name="right_wheel_collision">
+      <origin xyz="0 0 0" rpy="0 1.5707 1.5707" />
+      <geometry>
+        <cylinder radius="0.1" length="0.05" />
+      </geometry>
+    </collision>
+    <visual name="right_wheel_visual">
+      <origin xyz="0 0 0" rpy="0 1.5707 1.5707" />
+      <geometry>
+        <cylinder radius="0.1" length="0.05" />
+      </geometry>
+    </visual>
+  </link>
+  <joint type="continuous" name="right_wheel_hinge">
+    <origin xyz="0 -0.15 0" rpy="0 0 0" />
+    <child link="right_wheel" />
+    <parent link="chassis" />
+    <axis xyz="0 1 0" rpy="0 0 0" />
+    <limit effort="10000" velocity="1000" />
+    <dynamics damping="1.0" friction="1.0" />
+  </joint>
 </robot>

Commit message: camera and lidar added with relevant joints

File: src/my_robot/urdf/my_robot.xacro (robot description, xacro)
@@ -117,3 +117,53 @@
     <dynamics damping="1.0" friction="1.0" />
   </joint>
+  <link name="camera">
+    <inertial>
+      <mass value="0.1" />
+      <origin xyz="0 0 0" rpy="0 0 0" />
+      <inertia ixx="1e-6" ixy="0" ixz="0" iyy="1e-6" iyz="0" izz="1e-6" />
+    </inertial>
+    <collision name="camera_collision">
+      <origin xyz="0 0 0" rpy="0 0 0" />
+      <geometry>
+        <box size="0.05 0.05 0.05" />
+      </geometry>
+    </collision>
+    <visual name="camera_visual">
+      <origin xyz="0 0 0" rpy="0 0 0" />
+      <geometry>
+        <box size="0.05 0.05 0.05" />
+      </geometry>
+    </visual>
+  </link>
+  <joint type="fixed" name="camera_joint">
+    <origin xyz="0.2 0 0" rpy="0 0 0" />
+    <child link="camera" />
+    <parent link="chassis" />
+    <axis xyz="0 1 0" rpy="0 0 0" />
+  </joint>
+  <link name="hokuyo">
+    <inertial>
+      <mass value="1e-5" />
+      <origin xyz="0 0 0" rpy="0 0 0" />
+      <inertia ixx="1e-6" ixy="0" ixz="0" iyy="1e-6" iyz="0" izz="1e-6" />
+    </inertial>
+    <collision name="hokuyo_collision">
+      <origin xyz="0 0 0" rpy="0 0 0" />
+      <geometry>
+        <box size="0.1 0.1 0.1" />
+      </geometry>
+    </collision>
+    <visual name="hokuyo_visual">
+      <origin xyz="0 0 0" rpy="0 0 0" />
+      <geometry>
+        <mesh filename="package://my_robot/meshes/hokuyo.dae" />
+      </geometry>
+    </visual>
+  </link>
+  <joint type="fixed" name="hokuyo_joint">
+    <origin xyz="0.15 0 0.1" rpy="0 0 0" />
+    <child link="hokuyo" />
+    <parent link="chassis" />
+    <axis xyz="0 1 0" rpy="0 0 0" />
+  </joint>
 </robot>

Commit message: adding color, but does not work

File: src/my_robot/urdf/my_robot.xacro (robot description, xacro)
@@ -1,4 +1,13 @@
 <?xml version="1.0"?>
 <robot name="my_robot" xmlns:xacro="http://www.ros.org/wiki/xacro">
+  <material name="blue">
+    <color rgba="0 0 0.8 1" />
+  </material>
+  <material name="red">
+    <color rgba="0.8 0 0 1" />
+  </material>
+  <material name="green">
+    <color rgba="0 0.8 0 1" />
+  </material>
   <link name="robot_footprint"></link>
   <joint name="robot_footprint_joint" type="fixed">
@@ -13,8 +22,5 @@
       <origin xyz="0.0 0 0" rpy="0 0 0" />
       <inertia
-        ixx="0.1" ixy="0" ixz="0"
-        iyy="0.1" iyz="0"
-        izz="0.1"
-      />
+        ixx="0.1" ixy="0" ixz="0" iyy="0.1" iyz="0" izz="0.1" />
     </inertial>
     <collision name="collision">
@@ -29,4 +35,5 @@
         <box size="0.4 0.2 0.1" />
       </geometry>
+      <material name="blue" />
     </visual>
     <collision name="back_caster_collision">
@@ -60,8 +67,5 @@
       <origin xyz="0 0 0" rpy="0 1.5707 1.5707" />
       <inertia
-        ixx="0.1" ixy="0" ixz="0"
-        iyy="0.1" iyz="0"
-        izz="0.1"
-      />
+        ixx="0.1" ixy="0" ixz="0" iyy="0.1" iyz="0" izz="0.1" />
     </inertial>
     <collision name="left_wheel_collision">
@@ -91,8 +95,5 @@
       <origin xyz="0 0 0" rpy="0 1.5707 1.5707" />
       <inertia
-        ixx="0.1" ixy="0" ixz="0"
-        iyy="0.1" iyz="0"
-        izz="0.1"
-      />
+        ixx="0.1" ixy="0" ixz="0" iyy="0.1" iyz="0" izz="0.1" />
     </inertial>
     <collision name="right_wheel_collision">
@@ -134,4 +135,5 @@
         <box size="0.05 0.05 0.05" />
       </geometry>
+      <material name="red" />
     </visual>
   </link>

Commit message: at project "Go Chase It" concept 10, but camera and lidar sensors do not work correctly

File: src/my_robot/urdf/my_robot.xacro (robot description, xacro)
@@ -1,13 +1,5 @@
 <?xml version="1.0"?>
 <robot name="my_robot" xmlns:xacro="http://www.ros.org/wiki/xacro">
-  <material name="blue">
-    <color rgba="0 0 0.8 1" />
-  </material>
-  <material name="red">
-    <color rgba="0.8 0 0 1" />
-  </material>
-  <material name="green">
-    <color rgba="0 0.8 0 1" />
-  </material>
+  <xacro:include filename="$(find my_robot)/urdf/my_robot.gazebo" />
   <link name="robot_footprint"></link>
   <joint name="robot_footprint_joint" type="fixed">
@@ -24,5 +16,5 @@
         ixx="0.1" ixy="0" ixz="0" iyy="0.1" iyz="0" izz="0.1" />
     </inertial>
-    <collision name="collision">
+    <collision name="chassis_collision">
       <origin xyz="0 0 0" rpy="0 0 0" />
       <geometry>
@@ -35,5 +27,4 @@
         <box size="0.4 0.2 0.1" />
       </geometry>
-      <material name="blue" />
     </visual>
     <collision name="back_caster_collision">
@@ -135,5 +126,4 @@
         <box size="0.05 0.05 0.05" />
       </geometry>
-      <material name="red" />
     </visual>
   </link>
@@ -164,8 +154,20 @@
   </link>
   <joint type="fixed" name="hokuyo_joint">
-    <origin xyz="0.15 0 0.1" rpy="0 0 0" />
+    <origin xyz="0.15 0 0.08" rpy="0 0 0" />
     <child link="hokuyo" />
     <parent link="chassis" />
     <axis xyz="0 1 0" rpy="0 0 0" />
   </joint>
+  <gazebo reference="left_wheel">
+    <material>Gazebo/Green</material>
+  </gazebo>
+  <gazebo reference="right_wheel">
+    <material>Gazebo/Green</material>
+  </gazebo>
+  <gazebo reference="camera">
+    <material>Gazebo/Red</material>
+  </gazebo>
+  <gazebo reference="chassis">
+    <material>Gazebo/Blue</material>
+  </gazebo>
 </robot>
